File: io.kicad_sch (KiCad schematic)
At the start: 20 parts, among them J1 SLU0, J2 SLU1, SW4 Rate, U10 HD-6402_{B}, U11 AY-5-8116, U9 HD-6402_{A}, Y3 5.0688MHz

Commit message: get the GALs working with GALasm
Parts:
- U10: value HD-6402_{B} -> HD-6402
- U9: value HD-6402_{A} -> HD-6402
Changed lines of the file:
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@@
 			)
 		)
-		(property "Value" "HD-6402_{B}"
+		(property "Value" "HD-6402"
 			(at 143.1133 34.29 0)
 			(show_name no)
@@
 			)
 		)
-		(property "Value" "HD-6402_{A}"
+		(property "Value" "HD-6402"
 			(at 68.1833 34.29 0)
 			(show_name no)
