File: power.kicad_sch (KiCad schematic)
At the start: 20 parts, among them J3 5V, Q1 AO3401A, SW1 HMOD/BSEL, SW6 Power, U7 74HCT573, U8 22V10_{PWR}

Commit message: get the GALs working with GALasm
Connections:
- net GND: now also Q1.1 (G)
- net at R19.1: now also Q1.2 (S), SW6.3 (C); no longer Q1.1 (G)
Other:
- moved on the sheet: R19
Changed lines of the file:
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@@
 	(paper "A4")
 	(junction
+		(at 182.88 115.57)
+		(diameter 0)
+		(color 0 0 0 0)
+	)
+	(junction
 		(at 203.2 121.92)
 		(diameter 0)
@@
 	(junction
 		(at 182.88 143.51)
+		(diameter 0)
+		(color 0 0 0 0)
+	)
+	(junction
+		(at 190.5 121.92)
 		(diameter 0)
 		(color 0 0 0 0)
@@
 	(wire
 		(pts
-			(xy 190.5 118.11) (xy 190.5 121.92)
-		)
-		(stroke
-			(width 0)
-			(type default)
-		)
-	)
-	(wire
-		(pts
 			(xy 81.28 43.18) (xy 118.11 43.18)
 		)
@@
 	(wire
 		(pts
+			(xy 190.5 110.49) (xy 190.5 121.92)
+		)
+		(stroke
+			(width 0)
+			(type default)
+		)
+	)
+	(wire
+		(pts
 			(xy 55.88 55.88) (xy 55.88 58.42)
 		)
@@
 		(pts
 			(xy 81.28 111.76) (xy 93.98 111.76)
+		)
+		(stroke
+			(width 0)
+			(type default)
+		)
+	)
+	(wire
+		(pts
+			(xy 182.88 115.57) (xy 182.88 121.92)
 		)
 		(stroke
@@
 	(symbol
 		(lib_id "Device:R")
-		(at 190.5 114.3 0)
+		(at 186.69 121.92 90)
 		(unit 1)
 		(body_style 1)
@@
 		(fields_autoplaced yes)
 		(property "Reference" "R19"
-			(at 193.04 113.0299 0)
-			(show_name no)
-			(do_not_autoplace no)
-			(effects
-				(font
-					(size 1.27 1.27)
-				)
-				(justify left)
+			(at 186.69 115.57 90)
+			(show_name no)
+			(do_not_autoplace no)
+			(effects
+				(font
+					(size 1.27 1.27)
+				)
 			)
 		)
 		(property "Value" "100K"
-			(at 193.04 115.5699 0)
-			(show_name no)
-			(do_not_autoplace no)
-			(effects
-				(font
-					(size 1.27 1.27)
-				)
-				(justify left)
+			(at 186.69 118.11 90)
+			(show_name no)
+			(do_not_autoplace no)
+			(effects
+				(font
+					(size 1.27 1.27)
+				)
 			)
 		)
 		(property "Footprint" "J11Hack:R_Axial_DIN0207_L6.3mm_D2.5mm_P7.62mm_Horizontal"
-			(at 188.722 114.3 90)
+			(at 186.69 123.698 90)
 			(hide yes)
 			(show_name no)
@@
 		)
 		(property "Datasheet" ""
-			(at 190.5 114.3 0)
+			(at 186.69 121.92 0)
 			(hide yes)
 			(show_name no)
@@
 		)
 		(property "Description" "Resistor"
-			(at 190.5 114.3 0)
-			(hide yes)
-			(show_name no)
+			(at 186.69 121.92 0)
+			(hide yes)
+			(show_name no)
